File: SPEAR_PCB_Designs/LAN9252/untitled.kicad_sch (KiCad schematic)
At the start: 36 parts, among them J1 SM04B-GHS-TB, J3 SM04B-GHS-TB, T1 H1102NLT, T2 H1102NLT, U2 24FC512

Commit message: Changed it for real this time
Parts:
- removed T1, T2: H1102NLT, Transformer_SMD:Transformer_Pulse_H1100NL, symbol H1102NLT:H1102NLT
- added T1, T2: H1102NLT, SPEAR Footprints:XFMR_H1102NLT, symbol LAN9252 Symbols:H1102NLT
Connections:
- net GND: now also D2.1 (K), D3.1 (K); no longer D2.2 (A), D3.2 (A)
- net RXA N: now also T1.8
- net RXA P: now also T1.6
- net RXB N: now also T2.8
- net RXB P: now also T2.6
- net TXA N: now also T1.3
- net TXA P: now also T1.1
- net TXB N: now also T2.3
- net TXB P: now also T2.1
- net at R26.1: now also T2.15
- net at R20.2: now also D2.2 (A); no longer D2.1 (K)
- net at C23.1, R7.2: now also T1.2, T1.7
- net at R29.1: now also T1.10
- net at R27.1: now also T2.10
- net at J3.3 (Pin_3): now also T2.11
- net at J3.2 (Pin_2): now also T2.14
- net at J3.1 (Pin_1): now also T2.16
- net at C24.1, R12.2: now also T2.2, T2.7
- net at J3.4 (Pin_4): now also T2.9
- net at R21.2: now also D3.2 (A); no longer D3.1 (K)
- net at J1.1 (Pin_1): now also T1.16
- net at J1.2 (Pin_2): now also T1.14
- net at J1.3 (Pin_3): now also T1.11
- net at J1.4 (Pin_4): now also T1.9
- net at R28.1: now also T1.15
Other:
- moved on the sheet: D2, D3, J1

Commit message: Chris editted this.
Parts:
- C23, C24, C25, C26, C27: footprint Capacitor_SMD:C_0201_0603Metric -> Capacitor_SMD:C_0402_1005Metric
- D1, D2, D3: footprint LED_SMD:LED_0201_0603Metric -> LED_SMD:LED_0402_1005Metric
- J1: now in the parts list
- R10, R11, R12, R13, R14, R15, R16, R17, R18, R19, R20, R21, R26, R27, R28, R29, R3, R4, R5, R6, R7, R8, R9: footprint Resistor_SMD:R_0603_1608Metric -> Resistor_SMD:R_0402_1005Metric
- renumbered J3 to J2, U2 to U3
Other:
- moved on the sheet: C24, C26, C27, D1, D2, J2, R10, R11, R12, R13, R14, R15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
