File: SPEAR_PCB_Designs/Motor_Controller_Carrier_Board/board_connectors.kicad_sch (KiCad schematic)
At the start: 9 parts, among them J10 Conn_01x01_Socket, J11 Conn_01x01_Socket, J5 Conn_01x20_Socket, J6 Conn_01x20_Socket, J7 Conn_01x08_Socket, J8 Conn_01x01_Socket, J9 Conn_01x01_Socket

Commit message: Generated gerbers for carrier board with new buck converter layout
Parts:
- J10, J11, J8, J9: DigiKey_Part_Number 54-4637-0-00-15-00-00-03-0-ND -> ED1009-ND
Changed lines of the file:
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@@
 			)
 		)
-		(property "Datasheet" "https://www.mill-max.com/products/printed-circuit-board-pcb-pin/solder-mount-pcb-pin/4637"
+		(property "Datasheet" "https://www.mill-max.com/products/pin-receptacle/receptacle-with-standard-tail/0301/0301-1-15-15-47-27-10-0"
 			(at 218.44 100.33 0)
 			(effects
@@
 			)
 		)
-		(property "DigiKey_Part_Number" "54-4637-0-00-15-00-00-03-0-ND"
+		(property "DigiKey_Part_Number" "ED1009-ND"
 			(at 218.44 100.33 0)
 			(effects
@@
 			)
 		)
-		(property "Datasheet" "https://www.mill-max.com/products/printed-circuit-board-pcb-pin/solder-mount-pcb-pin/4637"
+		(property "Datasheet" "https://www.mill-max.com/products/pin-receptacle/receptacle-with-standard-tail/0301/0301-1-15-15-47-27-10-0"
 			(at 218.44 90.17 0)
 			(effects
@@
 			)
 		)
-		(property "DigiKey_Part_Number" "54-4637-0-00-15-00-00-03-0-ND"
+		(property "DigiKey_Part_Number" "ED1009-ND"
 			(at 218.44 90.17 0)
 			(effects
@@
 			)
 		)
-		(property "Datasheet" "https://www.mill-max.com/products/printed-circuit-board-pcb-pin/solder-mount-pcb-pin/4637"
+		(property "Datasheet" "https://www.mill-max.com/products/pin-receptacle/receptacle-with-standard-tail/0301/0301-1-15-15-47-27-10-0"
 			(at 218.44 85.09 0)
 			(effects
@@
 			)
 		)
-		(property "DigiKey_Part_Number" "54-4637-0-00-15-00-00-03-0-ND"
+		(property "DigiKey_Part_Number" "ED1009-ND"
 			(at 218.44 85.09 0)
 			(effects
@@
 			)
 		)
-		(property "Datasheet" "https://www.mill-max.com/products/printed-circuit-board-pcb-pin/solder-mount-pcb-pin/4637"
+		(property "Datasheet" "https://www.mill-max.com/products/pin-receptacle/receptacle-with-standard-tail/0301/0301-1-15-15-47-27-10-0"
 			(at 218.44 95.25 0)
 			(effects
@@
 			)
 		)
-		(property "DigiKey_Part_Number" "54-4637-0-00-15-00-00-03-0-ND"
+		(property "DigiKey_Part_Number" "ED1009-ND"
 			(at 218.44 95.25 0)
 			(effects
