File: SPEAR_PCB_Designs/SPEAR power junction/SPEAR power junction.kicad_sch (KiCad schematic)
At the start: 7 parts, among them J1 XT30PW-M, J2 XT30PW-M, J3 XT30PW-M, J5 XT90PW-M

Commit message: Updated Power junction design and fabrication folder
Parts:
- added F1: 3557-15, 3557-15:FUSE_3557-15, symbol 3557-15:3557-15
- added J4: SM02B-GHS-TB, SM02B-GHS-TB:CONN_SM02B-GHS_JST, symbol SM02B-GHS-TB:SM02B-GHS-TB
Connections:
- net GND: now also J4.1
- net Power: now also F1.1_1, F1.1_2
- new net: F1.2_1, F1.2_2, J4.2
