File: SPEAR_PCB_Designs/Stepper_Motor_Controller_Carrier_Board/Stepper_Motor_Controller_Carrier_Board.kicad_pcb (KiCad board)
At the start: 2 copper layers, 125.5 x 47 mm, 18 parts, among them J1 Conn_01x02_Pin, J2 Conn_01x02_Pin, J4 JST_S4B-XH-A-1, J5 Conn_01x02_Pin, J6 Conn_01x02_Pin, U1 AP63203WU

Commit message: Add files via upload
Parts:
- added C6: 10u, Capacitor_SMD:C_1210_3225Metric_Pad1.33x2.70mm_HandSolder, F.Cu at (116.9, 103.5)
- C1: footprint SPEAR_AP63203BuckConverter:CAP_FG20_TDK_C1 -> Capacitor_SMD:C_1210_3225Metric_Pad1.33x2.70mm_HandSolder
- C2, C4: footprint SPEAR_AP63203BuckConverter:CAP_FG22_TDK_C2_C4 -> Capacitor_SMD:C_1210_3225Metric_Pad1.33x2.70mm_HandSolder
- C3: footprint Capacitor_THT:C_Disc_D5.0mm_W2.5mm_P5.00mm -> Capacitor_SMD:C_1206_3216Metric
- moved F3 4.92 mm to (108.0, 103.1), turned to 90 degrees
- moved C4 4.59 mm to (110.6, 91.5)
- moved C2 2.18 mm to (127.1, 100.1)
- moved C1 1.98 mm to (116.9, 99.5)
- moved C3 1.75 mm to (116.5, 91.0)
Routing:
- net /BUCK_PWR: track 0.00 -> 4.06 mm
- net Net-(J1-Pin_2): track 65.9 -> 64.9 mm

Commit message: Add files via upload
Parts:
- removed C6: 10u, Capacitor_SMD:C_1210_3225Metric_Pad1.33x2.70mm_HandSolder
- added C5: 22uF, Motor_Controller_Carrier_Board:CAP_C3225X7R1C226M250AC, F.Cu at (126.0, 99.2)
- added G***: LOGO, SPEAR_Logos:spear_logo_10.0x10, B.Cu at (119.1, 85.5)
- C1: value 10u -> 10uF; footprint Capacitor_SMD:C_1210_3225Metric_Pad1.33x2.70mm_HandSolder -> Motor_Controller_Carrier_Board:CAPC3225X270N
- C2: value 22u -> 10uF; footprint Capacitor_SMD:C_1210_3225Metric_Pad1.33x2.70mm_HandSolder -> Motor_Controller_Carrier_Board:CAPC3225X270N
- C3: value 100n -> 150nF; footprint Capacitor_SMD:C_1206_3216Metric -> Motor_Controller_Carrier_Board:CAP_CC1206_YAG
- C4: value 22u -> 22uF; footprint Capacitor_SMD:C_1210_3225Metric_Pad1.33x2.70mm_HandSolder -> Motor_Controller_Carrier_Board:CAP_C3225X7R1C226M250AC
- F3: value Fuse -> 2A
- L1: value 3.9u -> 3.9uH
- U1: footprint Package_TO_SOT_SMD:TSOT-23-6 -> Motor_Controller_Carrier_Board:TSOT-23-6
- moved C4 19.3 mm to (126.0, 103.0)
- moved C2 11.4 mm to (116.2, 103.8), turned to 0 degrees
- moved F3 3.91 mm to (110.2, 99.8)
- moved L1 1.86 mm to (125.5, 91.5)
- moved C1 0.85 mm to (116.2, 100.0)
- moved U1 0.85 mm to (116.0, 96.0)
- moved C3 0.52 mm to (116.0, 91.2), turned to -90 degrees
Connections:
- net /SW renamed /Schematic/SW
- net Net-(U1-BST) renamed /Schematic/BST
- C1 pad 1: /BUCK_PWR -> /Schematic/BUCK_PWR
- C2 pad 1: +3.3V -> /Schematic/BUCK_PWR
- F3 pad 1: /BUCK_PWR -> /Schematic/BUCK_PWR
- U1 pad 2: /BUCK_PWR -> /Schematic/BUCK_PWR
- U1 pad 3: /BUCK_PWR -> /Schematic/BUCK_PWR
Routing:
- net /BUCK_PWR: track 4.06 -> 0.00 mm
- net /Schematic/BUCK_PWR: track 0.00 -> 4.02 mm
- net /Schematic/BST: track 5.55 -> 2.77 mm
- net Net-(J6-Pin_1): track 33.5 -> 31.0 mm
- net Net-(J1-Pin_2): track 64.9 -> 62.9 mm
- net /Schematic/SW: track 0.00 -> 1.25 mm
- net +3.3V: track 143.5 -> 142.3 mm
- net GND: vias 8 -> 6
- added copper zone on F.Cu, net /Schematic/BUCK_PWR
- removed copper zone on F.Cu, net /BUCK_PWR
Other:
- board text added: "Oliver Schneider Ronak Grover Henry Diep"

Commit message: Add files via upload
Parts:
- moved C5 1.58 mm to (187.5, 76.5)
- moved J5 1.00 mm to (195.0, 98.0)
Routing:
- net /DRIVER_PWR: track 51.5 -> 52.6 mm
- net Net-(J5-Pin_2): track 14.0 -> 15.0 mm
Changed lines of the file:
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@@
 	(footprint "Motor_Controller_Carrier_Board:CAP_UBY_18X20_NCH"
 		(layer "F.Cu")
-		(at 188 78 -90)
+		(at 187.5 76.5 -90)
 		(tags "URZ1H102MHD ")
 		(property "Reference" "C5"
@@
 	(footprint "Connector_AMASS:AMASS_XT30PW-M_1x02_P2.50mm_Horizontal"
 		(layer "F.Cu")
-		(at 194 98 -90)
+		(at 195 98 -90)
 		(descr "Connector XT30 Horizontal PCB Male, https://www.tme.eu/Document/6eb2005a51a52592b3f19e8a450c54c8/XT30PW-M.pdf")
 		(tags "RC Connector XT30")
@@
 	)
 	(segment
+		(start 140.215 75.955)
+		(end 142.27 73.9)
+		(width 0.3)
+		(layer "F.Cu")
+		(net 3)
+	)
+	(segment
 		(start 152.5 99.9)
 		(end 152.5 88.24)
@@
 	)
 	(segment
-		(start 182.75 75.75)
-		(end 204.15 75.75)
-		(width 0.3)
-		(layer "F.Cu")
-		(net 3)
-	)
-	(segment
 		(start 152.5 88.24)
 		(end 140.215 75.955)
@@
 	)
 	(segment
+		(start 182 75)
+		(end 203.4 75)
+		(width 0.3)
+		(layer "F.Cu")
+		(net 3)
+	)
+	(segment
+		(start 180.9 73.9)
+		(end 182 75)
+		(width 0.3)
+		(layer "F.Cu")
+		(net 3)
+	)
+	(segment
 		(start 113.25 95.6)
 		(end 113.8 95.05)
@@
 	)
 	(segment
-		(start 180.9 73.9)
-		(end 182.75 75.75)
-		(width 0.3)
-		(layer "F.Cu")
-		(net 3)
-	)
-	(segment
 		(start 152.5 99.9)
 		(end 153.6 101)
@@
 	)
 	(segment
-		(start 140.215 75.955)
-		(end 142.27 73.9)
-		(width 0.3)
+		(start 113.25 97.25)
+		(end 113.25 95.6)
+		(width 0.5)
 		(layer "F.Cu")
 		(net 3)
 	)
 	(segment
-		(start 113.25 97.25)
-		(end 113.25 95.6)
-		(width 0.5)
+		(start 203.4 75)
+		(end 204.15 75.75)
+		(width 0.3)
 		(layer "F.Cu")
 		(net 3)
@@
 	)
 	(segment
+		(start 184 83.5)
+		(end 184 80)
+		(width 3)
+		(layer "F.Cu")
+		(net 35)
+	)
+	(segment
+		(start 180.5 86.5)
+		(end 181 86.5)
+		(width 3)
+		(layer "F.Cu")
+		(net 35)
+	)
+	(segment
 		(start 165.8 76.4)
 		(end 175.9 86.5)
@@
 	)
 	(segment
-		(start 148.5 76.4)
-		(end 165.8 76.4)
+		(start 181 86.5)
+		(end 184 83.5)
 		(width 3)
 		(layer "F.Cu")
@@
 	(segment
 		(start 148.5 76.4)
-		(end 145.1 76.4)
-		(width 3.6)
+		(end 165.8 76.4)
+		(width 3)
 		(layer "F.Cu")
 		(net 35)
 	)
 	(segment
-		(start 181 86.5)
-		(end 188 79.5)
+		(start 184 80)
+		(end 187.149 76.851)
 		(width 3)
 		(layer "F.Cu")
@@
 	)
 	(segment
-		(start 188 79.5)
-		(end 188 78)
-		(width 3)
+		(start 148.5 76.4)
+		(end 145.1 76.4)
+		(width 3.6)
 		(layer "F.Cu")
 		(net 35)
 	)
 	(segment
-		(start 180.5 86.5)
-		(end 181 86.5)
+		(start 187.149 76.851)
+		(end 187.5 76.851)
 		(width 3)
 		(layer "F.Cu")
@@
 	)
 	(segment
-		(start 187 94.12)
-		(end 188.12 93)
+		(start 180.5 94.12)
+		(end 187 94.12)
 		(width 2)
 		(layer "F.Cu")
@@
 	)
 	(segment
-		(start 180.5 94.12)
-		(end 187 94.12)
+		(start 187 94.12)
+		(end 188.12 93)
 		(width 2)
 		(layer "F.Cu")
@@
 	(segment
 		(start 188.12 93)
-		(end 194 93)
+		(end 195 93)
 		(width 2)
 		(layer "F.Cu")

Commit message: Add files via upload
Parts:
- moved C5 0.71 mm to (188.0, 76.0)
Routing:
- net Net-(J6-Pin_1): track 31.0 -> 29.1 mm
- net /DRIVER_PWR: track 52.6 -> 53.7 mm
- net /ENC_B: track 148.8 -> 149.4 mm
Other:
- board size 125.5 x 47 mm -> 126 x 50.5 mm

Commit message: Add files via upload
Parts:
- removed the C5 at (188.0, 76.0)
- added REF**: MountingHole_3.2mm_M3, MountingHole:MountingHole_3.2mm_M3, F.Cu at (92.0, 119.5)
- moved J4 14.0 mm to (190.2, 84.2)
- moved J5 10.5 mm to (184.5, 97.5)
- moved J6 9.01 mm to (184.5, 112.0)
- moved REF** 4.46 mm to (170.5, 76.0)
- moved MDB2 2.68 mm to (153.7, 77.6)
Routing:
- net /ENC_B: track 149.4 -> 129.1 mm
- net /ENC_A: track 97.4 -> 80.6 mm
- net /DRIVER_PWR: track 53.7 -> 37.2 mm
- net +3.3V: track 142.3 -> 126.4 mm
- net /DMODE0: track 106.9 -> 98.5 mm
- net Net-(J5-Pin_2): track 15.0 -> 7.35 mm
- net Net-(J5-Pin_1): track 14.1 -> 7.03 mm
- net /DMODE1: track 98.0 -> 91.4 mm
- net Net-(J6-Pin_2): track 15.4 -> 8.82 mm
- net /DMODE2: track 89.8 -> 84.3 mm
- net Net-(J6-Pin_1): track 29.1 -> 24.1 mm
- net /CLK: track 72.9 -> 68.8 mm
- net /DIR: track 77.4 -> 74.8 mm
Other:
- board size 126 x 50.5 mm -> 113 x 49 mm
- board text added: "Oliver Schneider Ronak Grover Hazem Ammar Henry Diep"
- board text removed: "Oliver Schneider Ronak Grover Henry Diep"
