File: SPEAR_PCB_Designs/MP6550 Single Brushed DC Motor Driver Carrier/Motor_Controller_Carrier_Board.kicad_pcb (KiCad board)
At the start: 2 copper layers, 104 x 47 mm, 21 parts, among them J1 Conn_01x02_Pin, J2 Conn_01x02_Pin, J3 Conn_01x02_Pin, J4 Conn_01x04_Pin, U1 AP63203WU

Commit message: update
Parts:
- R1: footprint Resistor_SMD:R_01005_0402Metric -> Resistor_THT:R_Axial_DIN0207_L6.3mm_D2.5mm_P7.62mm_Horizontal
- moved REF** 22.6 mm to (171.1, 96.6)
- moved J3 15.2 mm to (159.8, 111.0)
- moved C6 11.4 mm to (148.5, 73.5)
- moved J4 7.83 mm to (172.7, 80.0)
- moved C7 7.10 mm to (173.4, 88.8)
- moved MDB1 5.56 mm to (152.2, 79.2)
- moved R1 3.87 mm to (158.2, 75.0)
Routing:
- net Net-(MDB1-ISET): track 4.20 -> 14.3 mm
- net +3.3V: track 117.7 -> 110.0 mm
- net /Schematic/ENC_A: track 70.0 -> 62.3 mm
- net GND: track 0.00 -> 6.86 mm
- net /Schematic/ENC_B: track 120.8 -> 114.4 mm
- net Net-(J3-Pin_1): track 51.8 -> 57.6 mm
- net Net-(MDB1-V3P3): track 32.7 -> 27.0 mm
- net Net-(J3-Pin_2): track 46.5 -> 51.4 mm
- net Net-(MDB1-VIN): track 35.4 -> 31.5 mm
- net /Schematic/PWM2: track 52.6 -> 48.8 mm
- net /Schematic/GPIO: track 53.8 -> 50.7 mm
- net /Schematic/PWM1: track 53.9 -> 51.4 mm
- net /Schematic/ADC: track 84.2 -> 83.3 mm
Other:
- board size 104 x 47 mm -> 98.5 x 47 mm

Commit message: updates
Parts:
- removed C6: 47uF, Motor_Controller_Carrier_Board:CAP_UBY_6.3X11_NCH
- removed C7: 0.47uF, Motor_Controller_Carrier_Board:CAP_UBY_18X20_NCH
- moved R1 27.7 mm to (153.0, 102.2), turned to -90 degrees
- moved REF** 27.0 mm to (152.0, 77.5)
- moved J4 10.5 mm to (162.2, 79.8)
- moved MDB1 3.92 mm to (154.6, 82.4)
- moved J3 2.78 mm to (158.6, 108.5)
Connections:
- MCB1 pad 22: /Schematic/PWM2 -> /Schematic/PWM1
- MCB1 pad 23: /Schematic/PWM1 -> /Schematic/PWM2
- MCB1 pad 31: /Schematic/CS -> unconnected-(MCB1-PB1-Pad31)
- MDB1 pad 6: Net-(MDB1-V3P3) -> GND
Routing:
- net Net-(J3-Pin_2): track 51.4 -> 5.37 mm
- net Net-(J3-Pin_1): track 57.6 -> 15.5 mm
- net /Schematic/PWM2: track 48.8 -> 82.3 mm
- net Net-(MDB1-V3P3): track 27.0 -> 0.00 mm
- net /Schematic/ADC: track 83.3 -> 110.2 mm
- net /Schematic/GPIO: track 50.7 -> 77.0 mm
- net /Schematic/PWM1: track 51.4 -> 75.3 mm
- net +3.3V: track 110.0 -> 99.2 mm
- net Net-(MDB1-VIN): track 31.5 -> 41.1 mm
- net Net-(MDB1-ISET): track 14.3 -> 7.07 mm
- net /Schematic/ENC_A: track 62.3 -> 56.4 mm
- net /Schematic/ENC_B: track 114.4 -> 118.8 mm
- net GND: track 6.86 -> 7.45 mm, vias 6 -> 9
Other:
- board size 98.5 x 47 mm -> 88.6 x 47.3 mm

Commit message: Update
Parts:
- removed MDB1: MP6550 Single Brushed DC Motor Driver Carrier, SPEAR_Boards:Motor_Driver_Board_2992
- added MDB3: Motor_Driver_Board_4733, SPEAR_Boards:Motor_Driver_Board_4733, F.Cu at (167.2, 84.9)
Routing:
- net GND: track 7.45 -> 0.10 mm, vias 9 -> 6
- net +3.3V: track 99.2 -> 102.6 mm

Commit message: Update Motor_Controller_Carrier_Board.kicad_pcb
Routing:
- net Net-(J3-Pin_2): track 5.37 -> 7.33 mm
- net Net-(J3-Pin_1): track 15.5 -> 14.5 mm
Changed lines of the file:
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@@
+	)
+	(segment
+		(start 158.35 103.24)
+		(end 158.61 103.5)
+		(width 0.3)
+		(layer "F.Cu")
+		(net 1)
 	)
 	(segment
 		(start 158.35 96.28)
-		(end 158.35 100.435558)
-		(width 0.3)
-		(layer "F.Cu")
-		(net 1)
-	)
-	(segment
-		(start 158.61 103.5)
-		(end 158.61 102.285558)
-		(width 3.6)
+		(end 158.35 103.24)
+		(width 0.3)
 		(layer "F.Cu")
 		(net 1)
@@
 		(layer "F.Cu")
 		(net 11)
-	)
-	(segment
-		(start 158.61 108.5)
-		(end 159.655558 108.5)
-		(width 3.6)
-		(layer "F.Cu")
-		(net 11)

Commit message: update
Parts:
- removed R1: 2kohm, Resistor_THT:R_Axial_DIN0207_L6.3mm_D2.5mm_P7.62mm_Horizontal
- moved J3 4.64 mm to (154.0, 108.0)
- moved REF** 1.00 mm to (153.0, 77.5)
Connections:
- MDB3 pad 11: Net-(MDB3-ISET) -> GND
Routing:
- net Net-(MDB3-ISET): track 7.07 -> 0.00 mm
- net Net-(J3-Pin_2): track 7.33 -> 8.87 mm
- net Net-(J3-Pin_1): track 14.5 -> 15.8 mm
Changed lines of the file:
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@@
 	(net 46 "Net-(MDB3-VIN)")
 	(net 47 "unconnected-(MDB3-VM-Pad1)")
-	(net 48 "Net-(MDB3-ISET)")
 	(footprint "SPEAR_Connectors:AMASS_XT30PW-M_1x02_P2.50mm_Horizontal_1"
 		(layer "F.Cu")
-		(at 158.61 108.5 -90)
+		(at 154 108 -90)
 		(descr "Connector XT30 Horizontal PCB Male, https://www.tme.eu/Document/6eb2005a51a52592b3f19e8a450c54c8/XT30PW-M.pdf")
 		(tags "RC Connector XT30")
@@
 	(footprint "MountingHole:MountingHole_3.2mm_M3"
 		(layer "F.Cu")
-		(at 152 77.5)
+		(at 153 77.5)
 		(descr "Mounting Hole 3.2mm, M3, no annular, generated by kicad-footprint-generator mountinghole.py")
 		(tags "mountinghole M3")
@@
 			(layers "*.Cu" "*.Mask")
 			(remove_unused_layers no)
-			(net 48 "Net-(MDB3-ISET)")
+			(net 2 "GND")
 			(pinfunction "ISET")
 			(pintype "input")
@@
 		)
 	)
-	(footprint "Resistor_THT:R_Axial_DIN0207_L6.3mm_D2.5mm_P7.62mm_Horizontal"
-		(layer "F.Cu")
-		(at 153 102.19 -90)
-		(descr "Resistor, Axial_DIN0207 series, Axial, Horizontal, pin pitch=7.62mm, 0.25W = 1/4W, length*diameter=6.3*2.5mm^2, http://cdn-reichelt.de/documents/datenblatt/B400/1_4W%23YAG.pdf")
-		(tags "Resistor Axial_DIN0207 series Axial Horizontal pin pitch 7.62mm 0.25W = 1/4W length 6.3mm diameter 2.5mm")
-		(property "Reference" "R1"
-			(at 3.81 -2.37 90)
-			(layer "F.SilkS")
-			(effects
-				(font
-					(size 1 1)
-					(thickness 0.15)
-				)
-			)
-		)
-		(property "Value" "2kohm"
-			(at 3.81 2.37 90)
-			(layer "F.Fab")
-			(effects
-				(font
-					(size 1 1)
-					(thickness 0.15)
-				)
-			)
-		)
-		(property "Datasheet" "https://www.digikey.com/en/products/detail/vishay-dale/PTF562K0000BYEB/2273678"
-			(at 0 0 90)
-			(layer "F.Fab")
-			(hide yes)
-			(effects
-				(font
-					(size 1.27 1.27)
-					(thickness 0.15)
-				)
-			)
-		)
-		(property "Description" "Resistor (moodel # PTF562K0000BYEB)"
-			(at 0 0 90)
-			(layer "F.Fab")
-			(hide yes)
-			(effects
-				(font
-					(size 1.27 1.27)
-					(thickness 0.15)
-				)
-			)
-		)
-		(property ki_fp_filters "R_*")
-		(sheetname "/Schematic/")
-		(sheetfile "schematic.kicad_sch")
-		(attr through_hole)
-		(fp_line
-			(start 0.54 1.37)
-			(end 7.08 1.37)
-			(stroke
-				(width 0.12)
-				(type solid)
-			)
-			(layer "F.SilkS")
-		)
-		(fp_line
-			(start 7.08 1.37)
-			(end 7.08 1.04)
-			(stroke
-				(width 0.12)
-				(type solid)
-			)
-			(layer "F.SilkS")
-		)
-		(fp_line
-			(start 0.54 1.04)
-			(end 0.54 1.37)
-			(stroke
-				(width 0.12)
-				(type solid)
-			)
-			(layer "F.SilkS")
-		)
-		(fp_line
-			(start 0.54 -1.04)
-			(end 0.54 -1.37)
-			(stroke
-				(width 0.12)
-				(type solid)
-			)
-			(layer "F.SilkS")
-		)
-		(fp_line
-			(start 0.54 -1.37)
-			(end 7.08 -1.37)
-			(stroke
-				(width 0.12)
-				(type solid)
-			)
-			(layer "F.SilkS")
-		)
-		(fp_line
-			(start 7.08 -1.37)
-			(end 7.08 -1.04)
-			(stroke
-				(width 0.12)
-				(type solid)
-			)
-			(layer "F.SilkS")
-		)
-		(fp_rect
-			(start -1.05 -1.5)
-			(end 8.67 1.5)
-			(stroke
-				(width 0.05)
-				(type solid)
-			)
-			(fill no)
-			(layer "F.CrtYd")
-		)
-		(fp_line
-			(start 0 0)
-			(end 0.66 0)
-			(stroke
-				(width 0.1)
-				(type solid)
-			)
-			(layer "F.Fab")
-		)
-		(fp_line
-			(start 7.62 0)
-			(end 6.96 0)
-			(stroke
-				(width 0.1)
-				(type solid)
-			)
-			(layer "F.Fab")
-		)
-		(fp_rect
-			(start 0.66 -1.25)
-			(end 6.96 1.25)
-			(stroke
-				(width 0.1)
-				(type solid)
-			)
-			(fill no)
-			(layer "F.Fab")
-		)
-		(fp_text user "${REFERENCE}"
-			(at 3.81 0 90)
-			(layer "F.Fab")
-			(effects
-				(font
-					(size 1 1)
-					(thickness 0.15)
-				)
-			)
-		)
-		(pad "1" thru_hole circle
-			(at 0 0 270)
-			(size 1.6 1.6)
-			(drill 0.8)
-			(layers "*.Cu" "*.Mask")
-			(remove_unused_layers no)
-			(net 48 "Net-(MDB3-ISET)")
-			(pintype "passive")
-		)
-		(pad "2" thru_hole circle
-			(at 7.62 0 270)
-			(size 1.6 1.6)
-			(drill 0.8)
-			(layers "*.Cu" "*.Mask")
-			(remove_unused_layers no)
-			(net 2 "GND")
-			(pintype "passive")
-		)
-		(embedded_fonts no)
-		(model "${KICAD9_3DMODEL_DIR}/Resistor_THT.3dshapes/R_Axial_DIN0207_L6.3mm_D2.5mm_P7.62mm_Horizontal.step"
-			(offset
-				(xyz 0 0 0)
-			)
-			(scale
-				(xyz 1 1 1)
-			)
-			(rotate
-				(xyz 0 0 0)
-			)
-		)
-	)
 	(footprint "Motor_Controller_Carrier_Board:FUSE_3557-15"
 		(layer "F.Cu")
@@
 	)
 	(gr_text "MOTOR"
-		(at 163.5 103 270)
+		(at 164.5 103 270)
 		(layer "F.SilkS")
 		(effects
@@
 	)
 	(gr_text "2992"
-		(at 156.81 112.1 0)
+		(at 152.2 111.6 0)
 		(layer "F.SilkS")
 		(effects
@@
 	)
 	(segment
-		(start 158.35 103.24)
-		(end 158.61 103.5)
+		(start 153.74 102.74)
+		(end 154 103)
+		(width 0.3)
+		(layer "F.Cu")
+		(net 1)
+	)
+	(segment
+		(start 158.33 96.29)
+		(end 158.33 98.67)
 		(width 0.3)
 		(layer "F.Cu")
@@
 	)
 	(segment
-		(start 158.35 96.28)
-		(end 158.35 103.24)
+		(start 158.33 98.67)
+		(end 154 103)
 		(width 0.3)
 		(layer "F.Cu")
@@
 	)
 	(segment
-		(start 160.89 106.22)
-		(end 160.89 96.28)
+		(start 160.87 96.29)
+		(end 160.87 101.13)
 		(width 0.3)
 		(layer "F.Cu")
@@
 	)
 	(segment
-		(start 157.699442 109.410558)
-		(end 158.61 108.5)
+		(start 153.089442 108.910558)
+		(end 154 108)
 		(width 0.3)
 		(layer "F.Cu")
@@
 	)
 	(segment
-		(start 158.61 108.5)
-		(end 160.89 106.22)
+		(start 160.87 101.13)
+		(end 154 108)
 		(width 0.3)
 		(layer "F.Cu")
@@
 		(net 46)
 	)
-	(segment
-		(start 155.81 96.28)
-		(end 155.81 99.38)
-		(width 0.3)
-		(layer "F.Cu")
-		(net 48)
-	)
-	(segment
-		(start 155.81 99.38)
-		(end 153 102.19)
-		(width 0.3)
-		(layer "F.Cu")
-		(net 48)
-	)
 	(zone
