File: SPEAR_PCB_Designs/MP6550 Single Brushed DC Motor Driver Carrier/board_connectors.kicad_sch (KiCad schematic)
At the start: 9 parts, among them J10 Conn_01x01_Socket, J11 Conn_01x01_Socket, J5 Conn_01x20_Socket, J6 Conn_01x20_Socket, J7 Conn_01x08_Socket, J8 Conn_01x01_Socket, J9 Conn_01x01_Socket

Commit message: updates
Parts:
- renumbered J11 to J?, J9 to J?, J5 to J?, J6 to J?, J8 to J?, J7 to J?, J10 to J?, MCB2 to MCB?, MDB2 to MDB?
Connections:
- net at J?.1 (Pin_1): now also MDB?.12 (SLP)
- net at MDB?.10 (IN2): now also J?.1 (Pin_1)
- net at MDB?.11 (IN2): now also J?.1 (Pin_1)
Other:
- moved on the sheet: J?
Changed lines of the file:
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@@
 	)
 	(junction
-		(at 217.17 100.33)
+		(at 217.17 99.06)
 		(diameter 0)
 		(color 0 0 0 0)
@@
 	(wire
 		(pts
-			(xy 215.9 90.17) (xy 218.44 90.17)
+			(xy 215.9 88.9) (xy 218.44 88.9)
 		)
 		(stroke
@@
 	(wire
 		(pts
-			(xy 215.9 95.25) (xy 218.44 95.25)
+			(xy 215.9 93.98) (xy 218.44 93.98)
 		)
 		(stroke
@@
 	(wire
 		(pts
-			(xy 217.17 100.33) (xy 218.44 100.33)
+			(xy 217.17 99.06) (xy 218.44 99.06)
 		)
 		(stroke
@@
 	(wire
 		(pts
-			(xy 215.9 100.33) (xy 217.17 100.33)
+			(xy 215.9 99.06) (xy 217.17 99.06)
 		)
 		(stroke
@@
 		(dnp no)
 		(fields_autoplaced yes)
-		(property "Reference" "#FLG06"
+		(property "Reference" "#FLG?"
 			(at 71.12 75.565 0)
 			(effects
@@
 	(symbol
 		(lib_id "Motor_Controller_Carrier_Board:Conn_01x01_Socket_Flipped")
-		(at 218.44 100.33 180)
+		(at 218.44 99.06 180)
 		(unit 1)
 		(exclude_from_sim no)
@@
 		(on_board yes)
 		(dnp no)
-		(property "Reference" "J11"
-			(at 225.806 100.33 0)
+		(property "Reference" "J?"
+			(at 225.806 99.06 0)
 			(effects
 				(font
@@
 		)
 		(property "Value" "Conn_01x01_Socket"
-			(at 239.776 100.33 0)
+			(at 239.776 99.06 0)
 			(effects
 				(font
@@
 		)
 		(property "Footprint" ""
-			(at 218.44 100.33 0)
+			(at 218.44 99.06 0)
 			(effects
 				(font
@@
 		)
 		(property "Datasheet" "https://www.mill-max.com/products/pin-receptacle/receptacle-with-standard-tail/0301/0301-1-15-15-47-27-10-0"
-			(at 218.44 100.33 0)
+			(at 218.44 99.06 0)
 			(effects
 				(font
@@
 		)
 		(property "Description" ""
-			(at 218.44 100.33 0)
+			(at 218.44 99.06 0)
 			(effects
 				(font
@@
 		)
 		(property "DigiKey_Part_Number" "ED1009-ND"
-			(at 218.44 100.33 0)
+			(at 218.44 99.06 0)
 			(effects
 				(font
@@
 		(dnp no)
 		(fields_autoplaced yes)
-		(property "Reference" "MDB2"
+		(property "Reference" "MDB?"
 			(at 203.2 77.47 0)
 			(effects
@@
 		(dnp no)
 		(fields_autoplaced yes)
-		(property "Reference" "#FLG04"
+		(property "Reference" "#FLG?"
 			(at 71.12 70.485 0)
 			(effects
@@
 	(symbol
 		(lib_id "Motor_Controller_Carrier_Board:Conn_01x01_Socket_Flipped")
-		(at 218.44 90.17 180)
+		(at 218.44 88.9 180)
 		(unit 1)
 		(exclude_from_sim no)
@@
 		(on_board yes)
 		(dnp no)
-		(property "Reference" "J9"
-			(at 225.806 90.17 0)
+		(property "Reference" "J?"
+			(at 225.806 88.9 0)
 			(effects
 				(font
@@
 		)
 		(property "Value" "Conn_01x01_Socket"
-			(at 239.776 90.17 0)
+			(at 239.776 88.9 0)
 			(effects
 				(font
@@
 		)
 		(property "Footprint" ""
-			(at 218.44 90.17 0)
+			(at 218.44 88.9 0)
 			(effects
 				(font
@@
 		)
 		(property "Datasheet" "https://www.mill-max.com/products/pin-receptacle/receptacle-with-standard-tail/0301/0301-1-15-15-47-27-10-0"
-			(at 218.44 90.17 0)
+			(at 218.44 88.9 0)
 			(effects
 				(font
@@
 		)
 		(property "Description" ""
-			(at 218.44 90.17 0)
+			(at 218.44 88.9 0)
 			(effects
 				(font
@@
 		)
 		(property "DigiKey_Part_Number" "ED1009-ND"
-			(at 218.44 90.17 0)
+			(at 218.44 88.9 0)
 			(effects
 				(font
@@
 		(dnp no)
 		(fields_autoplaced yes)
-		(property "Reference" "#FLG08"
+		(property "Reference" "#FLG?"
 			(at 189.23 81.915 0)
 			(effects
@@
 		(on_board yes)
 		(dnp no)
-		(property "Reference" "J5"
+		(property "Reference" "J?"
 			(at 54.61 89.154 0)
 			(effects
@@
 		(on_board yes)
 		(dnp no)
-		(property "Reference" "J6"
+		(property "Reference" "J?"
 			(at 133.35 89.154 0)
 			(effects
@@
 		(dnp no)
 		(fields_autoplaced yes)
-		(property "Reference" "#FLG05"
+		(property "Reference" "#FLG?"
 			(at 71.12 73.025 0)
 			(effects
@@
 		(dnp no)
 		(fields_autoplaced yes)
-		(property "Reference" "#FLG09"
+		(property "Reference" "#FLG?"
 			(at 217.17 83.185 0)
 			(effects
@@
 		(on_board yes)
 		(dnp no)
-		(property "Reference" "J8"
+		(property "Reference" "J?"
 			(at 225.806 85.09 0)
 			(effects
@@
 		(on_board yes)
 		(dnp no)
-		(property "Reference" "J7"
+		(property "Reference" "J?"
 			(at 171.196 89.662 0)
 			(effects
@@
 		(dnp no)
 		(fields_autoplaced yes)
-		(property "Reference" "MCB2"
+		(property "Reference" "MCB?"
 			(at 93.98 63.5 0)
 			(effects
@@
 		(dnp no)
 		(fields_autoplaced yes)
-		(property "Reference" "#FLG07"
+		(property "Reference" "#FLG?"
 			(at 71.12 67.945 0)
 			(effects
@@
 	(symbol
 		(lib_id "Motor_Controller_Carrier_Board:Conn_01x01_Socket_Flipped")
-		(at 218.44 95.25 180)
+		(at 218.44 93.98 180)
 		(unit 1)
 		(exclude_from_sim no)
@@
 		(on_board yes)
 		(dnp no)
-		(property "Reference" "J10"
-			(at 225.806 95.25 0)
+		(property "Reference" "J?"
+			(at 225.806 93.98 0)
 			(effects
 				(font
@@
 		)
 		(property "Value" "Conn_01x01_Socket"
-			(at 239.776 95.25 0)
+			(at 239.776 93.98 0)
 			(effects
 				(font
@@
 		)
 		(property "Footprint" ""
-			(at 218.44 95.25 0)
+			(at 218.44 93.98 0)
 			(effects
 				(font
@@
 		)
 		(property "Datasheet" "https://www.mill-max.com/products/pin-receptacle/receptacle-with-standard-tail/0301/0301-1-15-15-47-27-10-0"
-			(at 218.44 95.25 0)
+			(at 218.44 93.98 0)
 			(effects
 				(font
@@
 		)
 		(property "Description" ""
-			(at 218.44 95.25 0)
+			(at 218.44 93.98 0)
 			(effects
 				(font
@@
 		)
 		(property "DigiKey_Part_Number" "ED1009-ND"
-			(at 218.44 95.25 0)
+			(at 218.44 93.98 0)
 			(effects
 				(font
@@
 	(symbol
 		(lib_id "Motor_Controller_Carrier_Board:PWR_FLAG_Inline")
-		(at 217.17 100.33 0)
+		(at 217.17 99.06 0)
 		(unit 1)
 		(exclude_from_sim no)
@@
 		(dnp no)
 		(fields_autoplaced yes)
-		(property "Reference" "#FLG010"
-			(at 217.17 98.425 0)
+		(property "Reference" "#FLG?"
+			(at 217.17 97.155 0)
 			(effects
 				(font
@@
 		)
 		(property "Value" "PWR_FLAG_Inline"
-			(at 217.17 96.52 0)
+			(at 217.17 95.25 0)
 			(effects
 				(font
@@
 		)
 		(property "Footprint" ""
-			(at 217.17 100.33 0)
+			(at 217.17 99.06 0)
 			(effects
 				(font
@@
 		)
 		(property "Datasheet" "~"
-			(at 217.17 100.33 0)
+			(at 217.17 99.06 0)
 			(effects
 				(font
@@
 		)
 		(property "Description" "Special symbol for telling ERC where power comes from"
-			(at 217.17 100.33 0)
-			(effects
-				(font
+			(at 217.17 99.06 0)
+			(effects
+				(font

Commit message: update
Parts:
- gave numbers to parts that had none: 9
Changed lines of the file:
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@@
 		(dnp no)
 		(fields_autoplaced yes)
-		(property "Reference" "#FLG?"
+		(property "Reference" "#FLG06"
 			(at 71.12 75.565 0)
 			(effects
@@
 		(on_board yes)
 		(dnp no)
-		(property "Reference" "J?"
+		(property "Reference" "J11"
 			(at 225.806 99.06 0)
 			(effects
@@
 		(dnp no)
 		(fields_autoplaced yes)
-		(property "Reference" "MDB?"
+		(property "Reference" "MDB2"
 			(at 203.2 77.47 0)
 			(effects
@@
 		(dnp no)
 		(fields_autoplaced yes)
-		(property "Reference" "#FLG?"
+		(property "Reference" "#FLG04"
 			(at 71.12 70.485 0)
 			(effects
@@
 		(on_board yes)
 		(dnp no)
-		(property "Reference" "J?"
+		(property "Reference" "J9"
 			(at 225.806 88.9 0)
 			(effects
@@
 		(dnp no)
 		(fields_autoplaced yes)
-		(property "Reference" "#FLG?"
+		(property "Reference" "#FLG08"
 			(at 189.23 81.915 0)
 			(effects
@@
 		(on_board yes)
 		(dnp no)
-		(property "Reference" "J?"
+		(property "Reference" "J5"
 			(at 54.61 89.154 0)
 			(effects
@@
 		(on_board yes)
 		(dnp no)
-		(property "Reference" "J?"
+		(property "Reference" "J6"
 			(at 133.35 89.154 0)
 			(effects
@@
 		(dnp no)
 		(fields_autoplaced yes)
-		(property "Reference" "#FLG?"
+		(property "Reference" "#FLG05"
 			(at 71.12 73.025 0)
 			(effects
@@
 		(dnp no)
 		(fields_autoplaced yes)
-		(property "Reference" "#FLG?"
+		(property "Reference" "#FLG09"
 			(at 217.17 83.185 0)
 			(effects
@@
 		(on_board yes)
 		(dnp no)
-		(property "Reference" "J?"
+		(property "Reference" "J8"
 			(at 225.806 85.09 0)
 			(effects
@@
 		(on_board yes)
 		(dnp no)
-		(property "Reference" "J?"
+		(property "Reference" "J7"
 			(at 171.196 89.662 0)
 			(effects
@@
 		(dnp no)
 		(fields_autoplaced yes)
-		(property "Reference" "MCB?"
+		(property "Reference" "MCB2"
 			(at 93.98 63.5 0)
 			(effects
@@
 		(dnp no)
 		(fields_autoplaced yes)
-		(property "Reference" "#FLG?"
+		(property "Reference" "#FLG07"
 			(at 71.12 67.945 0)
 			(effects
@@
 		(on_board yes)
 		(dnp no)
-		(property "Reference" "J?"
+		(property "Reference" "J10"
 			(at 225.806 93.98 0)
 			(effects
@@
 		(dnp no)
 		(fields_autoplaced yes)
-		(property "Reference" "#FLG?"
+		(property "Reference" "#FLG010"
 			(at 217.17 97.155 0)
 			(effects
