File: SPEAR_PCB_Designs/MP6550 Single Brushed DC Motor Driver Carrier/schematic.kicad_sch (KiCad schematic)
At the start: 19 parts, among them J1 Conn_01x02_Pin, J2 Conn_01x02_Pin, J3 Conn_01x02_Pin, J4 Conn_01x04_Pin, U1 AP63203WU

Commit message: update
Parts:
- R1: footprint Resistor_SMD:R_01005_0402Metric -> Resistor_THT:R_Axial_DIN0207_L6.3mm_D2.5mm_P7.62mm_Horizontal
Changed lines of the file:
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@@
 			)
 		)
-		(property "Footprint" "Resistor_SMD:R_01005_0402Metric"
+		(property "Footprint" "Resistor_THT:R_Axial_DIN0207_L6.3mm_D2.5mm_P7.62mm_Horizontal"
 			(at 189.738 137.16 90)
 			(effects
@@
 			)
 		)
-		(property "Datasheet" "~"
+		(property "Datasheet" "https://www.digikey.com/en/products/detail/vishay-dale/PTF562K0000BYEB/2273678"
 			(at 187.96 137.16 0)
 			(effects
@@
 			)
 		)
-		(property "Description" "Resistor"
+		(property "Description" "Resistor (moodel # PTF562K0000BYEB)"
 			(at 187.96 137.16 0)
 			(effects

Commit message: updates
Parts:
- removed C6: 47uF, Motor_Controller_Carrier_Board:CAP_UBY_6.3X11_NCH, symbol Device:C
- removed C7: 0.47uF, Motor_Controller_Carrier_Board:CAP_UBY_18X20_NCH, symbol Device:C
- renumbered F2 to F1, F3 to F2, F1 to F3, J2 to J1, J1 to J2
Connections:
- net GND: now also MDB1.6 (V3P3)
- net PWM1: now also MCB1.22 (PC7); no longer MCB1.23 (PC8)
- net PWM2: now also MCB1.23 (PC8); no longer MCB1.22 (PC7)
- net CS: no longer names the net of MCB1.31 (PB1)
- no-connect marks 28 -> 30
Other:
- note added: "Buck converter"

Commit message: Update
Parts:
- removed MDB1: MP6550 Single Brushed DC Motor Driver Carrier, SPEAR_Boards:Motor_Driver_Board_2992, symbol SPEAR_Boards:Motor_Driver_Board_2992
- added MDB1: Motor_Driver_Board_4733, SPEAR_Boards:Motor_Driver_Board_4733, symbol SPEAR_Boards:Motor_Driver_Board_4733
- MCB1: now in the parts list
Connections:
- net ADC: now also MDB1.5 (VISEN)
- net GND: now also MDB1.12 (V3P3), MDB1.2 (GND), MDB1.8 (GND)
- net GPIO: now also MDB1.6 (SLEEP)
- net PWM1: now also MDB1.3 (IN2)
- net PWM2: now also MDB1.4 (IN1)
- net at J3.1 (Pin_1): now also MDB1.9 (OUT2)
- net at J3.2 (Pin_2): now also MDB1.10 (OUT1)
- net at F3.2_1, F3.2_2: now also MDB1.7 (VIN)
- net at R1.1: now also MDB1.11 (ISET)
- no-connect marks 30 -> 31
Other:
- moved on the sheet: J3, R1

Commit message: update
Parts:
- removed R1: 2kohm, Resistor_THT:R_Axial_DIN0207_L6.3mm_D2.5mm_P7.62mm_Horizontal, symbol Device:R
- renumbered F3 to F1, F1 to F2, F2 to F3, J2 to J1, J1 to J2, MDB1 to MDB3
Connections:
- net GND: now also MDB3.11 (ISET)
Changed lines of the file:
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@@
 	(wire
 		(pts
-			(xy 226.06 137.16) (xy 226.06 144.78)
-		)
-		(stroke
-			(width 0)
-			(type default)
-		)
-	)
-	(wire
-		(pts
 			(xy 73.66 81.28) (xy 73.66 82.55)
 		)
@@
 	(wire
 		(pts
-			(xy 226.06 118.11) (xy 226.06 129.54)
+			(xy 226.06 118.11) (xy 226.06 144.78)
 		)
 		(stroke
@@
 		(on_board yes)
 		(dnp no)
-		(property "Reference" "#PWR0106"
+		(property "Reference" "#PWR014"
 			(at 158.75 52.07 0)
 			(effects
@@
 				)
 			)
+			(project "Motor_Controller_Carrier_Board"
+				(path "/f3c97344-c35a-4a43-a333-44ea37de3455/8e110934-84f0-49b8-afcb-71c9a138826c"
+					(reference "MCB1")
+					(unit 1)
+				)
+			)
 		)
 	)
@@
 		(on_board yes)
 		(dnp no)
-		(property "Reference" "#PWR0103"
+		(property "Reference" "#PWR01"
 			(at 106.68 152.4 0)
 			(effects
@@
 		(on_board yes)
 		(dnp no)
-		(property "Reference" "#PWR0116"
+		(property "Reference" "#PWR08"
 			(at 215.9 116.84 0)
 			(effects
@@
 		(on_board yes)
 		(dnp no)
-		(property "Reference" "#PWR0107"
+		(property "Reference" "#PWR010"
 			(at 158.75 41.91 0)
 			(effects
@@
 		(on_board yes)
 		(dnp no)
-		(property "Reference" "#PWR0108"
+		(property "Reference" "#PWR011"
 			(at 158.75 46.99 0)
 			(effects
@@
 		(on_board yes)
 		(dnp no)
-		(property "Reference" "#PWR0110"
+		(property "Reference" "#PWR04"
 			(at 55.88 93.98 0)
 			(effects
@@
 	)
 	(symbol
-		(lib_id "Device:R")
-		(at 226.06 133.35 0)
-		(unit 1)
-		(exclude_from_sim no)
-		(in_bom yes)
-		(on_board yes)
-		(dnp no)
-		(fields_autoplaced yes)
-		(property "Reference" "R1"
-			(at 228.6 132.0799 0)
-			(effects
-				(font
-					(size 1.27 1.27)
-				)
-				(justify left)
-			)
-		)
-		(property "Value" "2kohm"
-			(at 228.6 134.6199 0)
-			(effects
-				(font
-					(size 1.27 1.27)
-				)
-				(justify left)
-			)
-		)
-		(property "Footprint" "Resistor_THT:R_Axial_DIN0207_L6.3mm_D2.5mm_P7.62mm_Horizontal"
-			(at 224.282 133.35 90)
-			(effects
-				(font
-					(size 1.27 1.27)
-				)
-				(hide yes)
-			)
-		)
-		(property "Datasheet" "https://www.digikey.com/en/products/detail/vishay-dale/PTF562K0000BYEB/2273678"
-			(at 226.06 133.35 0)
-			(effects
-				(font
-					(size 1.27 1.27)
-				)
-				(hide yes)
-			)
-		)
-		(property "Description" "Resistor (moodel # PTF562K0000BYEB)"
-			(at 226.06 133.35 0)
-			(effects
-				(font
-					(size 1.27 1.27)
-				)
-				(hide yes)
-			)
-		)
-		(pin "1"
-		)
-		(pin "2"
-		)
-		(instances
-			(project ""
-				(path "/3ea9b895-1707-441b-a55c-91c8f6d35536"
-					(reference "R1")
-					(unit 1)
-				)
-			)
-			(project "Motor_Controller_Carrier_Board"
-				(path "/f3c97344-c35a-4a43-a333-44ea37de3455/8e110934-84f0-49b8-afcb-71c9a138826c"
-					(reference "R1")
-					(unit 1)
-				)
-			)
-		)
-	)
-	(symbol
 		(lib_id "power:GND")
 		(at 116.84 86.36 0)
@@
 		(on_board yes)
 		(dnp no)
-		(property "Reference" "#PWR0109"
+		(property "Reference" "#PWR02"
 			(at 116.84 92.71 0)
 			(effects
@@
 		(on_board yes)
 		(dnp no)
-		(property "Reference" "J2"
+		(property "Reference" "J1"
 			(at 72.136 148.59 0)
 			(effects
@@
 		(dnp no)
 		(fields_autoplaced yes)
-		(property "Reference" "#PWR0104"
+		(property "Reference" "#PWR015"
 			(at 93.98 157.48 0)
 			(effects
@@
 		(dnp no)
 		(fields_autoplaced yes)
-		(property "Reference" "#FLG0104"
+		(property "Reference" "#FLG011"
 			(at 116.84 61.595 0)
 			(effects
@@
 		(on_board yes)
 		(dnp no)
-		(property "Reference" "#PWR0102"
+		(property "Reference" "#PWR07"
 			(at 82.55 129.54 0)
 			(effects
@@
 		(dnp no)
 		(fields_autoplaced yes)
-		(property "Reference" "MDB1"
+		(property "Reference" "MDB3"
 			(at 199.39 101.6 0)
 			(effects
@@
 		(on_board yes)
 		(dnp no)
-		(property "Reference" "#FLG0101"
+		(property "Reference" "#FLG01"
 			(at 99.695 125.73 0)
 			(effects
@@
 		(dnp no)
 		(fields_autoplaced yes)
-		(property "Reference" "F2"
+		(property "Reference" "F3"
 			(at 100.33 133.3499 0)
 			(effects
@@
 		(dnp no)
 		(fields_autoplaced yes)
-		(property "Reference" "#PWR0114"
+		(property "Reference" "#PWR013"
 			(at 232.41 64.77 0)
 			(effects
@@
 		(on_board yes)
 		(dnp no)
-		(property "Reference" "#PWR0115"
+		(property "Reference" "#PWR012"
 			(at 238.76 66.04 0)
 			(effects
@@
 		(on_board yes)
 		(dnp no)
-		(property "Reference" "#PWR0113"
+		(property "Reference" "#PWR05"
 			(at 179.07 116.84 0)
 			(effects
@@
 		(on_board yes)
 		(dnp no)
-		(property "Reference" "J1"
+		(property "Reference" "J2"
 			(at 72.136 120.65 0)
 			(effects
@@
 		(on_board yes)
 		(dnp no)
-		(property "Reference" "#PWR0111"
+		(property "Reference" "#PWR03"
 			(at 41.91 93.98 0)
 			(effects
@@
 		(on_board yes)
 		(dnp no)
-		(property "Reference" "#PWR02"
+		(property "Reference" "#PWR0102"
 			(at 226.06 151.13 0)
 			(effects
@@
 		(on_board yes)
 		(dnp no)
-		(property "Reference" "F1"
+		(property "Reference" "F2"
 			(at 85.09 133.35 90)
 			(effects
@@
 		(on_board yes)
 		(dnp no)
-		(property "Reference" "F3"
+		(property "Reference" "F1"
 			(at 110.49 154.94 0)
 			(effects
@@
 		(dnp no)
 		(fields_autoplaced yes)
-		(property "Reference" "#PWR0112"
+		(property "Reference" "#PWR06"
 			(at 215.9 140.97 0)
 			(effects
@@
 		(dnp no)
 		(fields_autoplaced yes)
-		(property "Reference" "#FLG0102"
+		(property "Reference" "#FLG03"
 			(at 121.92 146.685 0)
 			(effects
