File: SPEAR_PCB_Designs/DriveControllerCarrier/DriveControllerCarrier.kicad_pcb (KiCad board)
At the start: 2 copper layers, 104 x 47 mm, 19 parts, among them J1 Conn_01x02_Pin, J2 Conn_01x02_Pin, J3 Conn_01x02_Pin, J4 Conn_01x04_Pin, U1 AP63203WU

Commit message: Routed traces for unconnected pins on stepper motor driver and did some organizing
Parts:
- C1, C2: footprint Motor_Controller_Carrier_Board:CAPC3225X270N -> SPEAR_MotorControllerCarrier:CAPC3225X270N
- C3: footprint Motor_Controller_Carrier_Board:CAP_CC1206_YAG -> SPEAR_MotorControllerCarrier:CAP_CC1206_YAG
- C4, C5: footprint Motor_Controller_Carrier_Board:CAP_C3225X7R1C226M250AC -> SPEAR_MotorControllerCarrier:CAP_C3225X7R1C226M250AC
- C6: footprint Motor_Controller_Carrier_Board:CAP_UBY_18X20_NCH -> SPEAR_MotorControllerCarrier:CAP_UBY_18X20_NCH
- F1: footprint Motor_Controller_Carrier_Board:FUSE_3557-10 -> SPEAR_MotorControllerCarrier:FUSE_3557-10
- F2: footprint Motor_Controller_Carrier_Board:FUSE_3557-15 -> SPEAR_MotorControllerCarrier:FUSE_3557-15
- F3: footprint Motor_Controller_Carrier_Board:FUS_LITTELFUSE_392_LTF -> SPEAR_MotorControllerCarrier:FUS_LITTELFUSE_392_LTF
- U1: footprint Motor_Controller_Carrier_Board:TSOT-23-6 -> SPEAR_MotorControllerCarrier:TSOT-23-6
Changed lines of the file:
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@@
 		)
 		(embedded_fonts no)
-		(model "${SPEAR_PCB_2026_DIR}/SPEAR_3D_Models/SPEAR_Motor_Controller_Carrier_Board/XT30PW-M.stp"
+		(model "${SPEAR_PCB_2026_DIR}/SPEAR_3D_Models/SPEAR_MotorControllerCarrier/XT30PW-M.stp"
 			(offset
 				(xyz -2.5 4.1 2.5)
@@
 			(layer "F.CrtYd")
 		)
+		(fp_text user "${REFERENCE}"
+			(at 0 0 0)
+			(layer "F.Fab")
+			(effects
+				(font
+					(size 1 1)
+					(thickness 0.15)
+				)
+			)
+		)
 		(pad "" np_thru_hole circle
 			(at 0 0)
@@
 		(embedded_fonts no)
 	)
-	(footprint "Motor_Controller_Carrier_Board:CAPC3225X270N"
+	(footprint "SPEAR_MotorControllerCarrier:CAPC3225X270N"
 		(layer "F.Cu")
 		(at 113.75 100.98675)
@@
 		)
 		(embedded_fonts no)
-		(model "${SPEAR_PCB_2026_DIR}/SPEAR_3D_Models/SPEAR_Motor_Controller_Carrier_Board/GCM32EC71H106KA03L.step"
+		(model "${SPEAR_PCB_2026_DIR}/SPEAR_3D_Models/SPEAR_MotorControllerCarrier/GCM32EC71H106KA03L.step"
 			(offset
 				(xyz 0 -1.35 1.3)
@@
 		)
 	)
-	(footprint "Motor_Controller_Carrier_Board:TSOT-23-6"
+	(footprint "SPEAR_MotorControllerCarrier:TSOT-23-6"
 		(layer "F.Cu")
 		(at 113.5 93.23675)
@@
 		)
 	)
-	(footprint "Motor_Controller_Carrier_Board:FUS_LITTELFUSE_392_LTF"
+	(footprint "SPEAR_MotorControllerCarrier:FUS_LITTELFUSE_392_LTF"
 		(layer "F.Cu")
 		(at 107.7 97.08675 90)
@@
 		)
 		(embedded_fonts no)
-		(model "${SPEAR_PCB_2026_DIR}/SPEAR_3D_Models/SPEAR_Motor_Controller_Carrier_Board/FUS_LITTELFUSE_392_LTF.step"
+		(model "${SPEAR_PCB_2026_DIR}/SPEAR_3D_Models/SPEAR_MotorControllerCarrier/FUS_LITTELFUSE_392_LTF.step"
 			(offset
-				(xyz 0.5 0 0)
+				(xyz 0.4 0 0)
 			)
 			(scale
@@
 		)
 		(embedded_fonts no)
-		(model "${SPEAR_PCB_2026_DIR}/SPEAR_3D_Models/SPEAR_Motor_Controller_Carrier_Board/WE-LHMI_1040.stp"
+		(model "${SPEAR_PCB_2026_DIR}/SPEAR_3D_Models/SPEAR_MotorControllerCarrier/WE-LHMI_1040.stp"
 			(offset
 				(xyz 0 0 0)
@@
 		)
 		(embedded_fonts no)
-		(model "${SPEAR_PCB_2026_DIR}/SPEAR_3D_Models/SPEAR_Motor_Controller_Carrier_Board/61302011821.stp"
+		(model "${SPEAR_PCB_2026_DIR}/SPEAR_3D_Models/SPEAR_MotorControllerCarrier/61302011821.stp"
 			(offset
 				(xyz 3 -26.3 4.3)
@@
 			)
 		)
-		(model "${SPEAR_PCB_2026_DIR}/SPEAR_3D_Models/SPEAR_Motor_Controller_Carrier_Board/61302011821.stp"
+		(model "${SPEAR_PCB_2026_DIR}/SPEAR_3D_Models/SPEAR_MotorControllerCarrier/61302011821.stp"
 			(offset
 				(xyz 41 -28.9 4.3)
@@
 		)
 		(embedded_fonts no)
-		(model "${SPEAR_PCB_2026_DIR}/SPEAR_3D_Models/SPEAR_Motor_Controller_Carrier_Board/g2-high-power-motor-driver-md31a.step"
+		(model "${SPEAR_PCB_2026_DIR}/SPEAR_3D_Models/SPEAR_MotorControllerCarrier/g2-high-power-motor-driver-md31a.step"
 			(offset
 				(xyz -0.1 -20.25 11.9)
@@
 			)
 		)
-		(model "${SPEAR_PCB_2026_DIR}/SPEAR_3D_Models/SPEAR_Motor_Controller_Carrier_Board/61300811821.stp"
+		(model "${SPEAR_PCB_2026_DIR}/SPEAR_3D_Models/SPEAR_MotorControllerCarrier/61300811821.stp"
 			(offset
 				(xyz 1.2 -10.2 4.3)
@@
 			)
 		)
-		(model "${SPEAR_PCB_2026_DIR}/SPEAR_3D_Models/SPEAR_Motor_Controller_Carrier_Board/61300811121.stp"
+		(model "${SPEAR_PCB_2026_DIR}/SPEAR_3D_Models/SPEAR_MotorControllerCarrier/61300811121.stp"
 			(offset
 				(xyz 1.2 -10.1 9.9)
@@
 			)
 		)
-		(model "${SPEAR_PCB_2026_DIR}/SPEAR_3D_Models/SPEAR_Motor_Controller_Carrier_Board/mill-max-4637-0-00-15-00-00-03-0.step"
+		(model "${SPEAR_PCB_2026_DIR}/SPEAR_3D_Models/SPEAR_MotorControllerCarrier/mill-max-4637-0-00-15-00-00-03-0.step"
 			(offset
 				(xyz 29.1 -1.2 14.6)
@@
 			)
 		)
-		(model "${SPEAR_PCB_2026_DIR}/SPEAR_3D_Models/SPEAR_Motor_Controller_Carrier_Board/mill-max-4637-0-00-15-00-00-03-0.step"
+		(model "${SPEAR_PCB_2026_DIR}/SPEAR_3D_Models/SPEAR_MotorControllerCarrier/mill-max-4637-0-00-15-00-00-03-0.step"
 			(offset
 				(xyz 29.1 -6.3 14.6)
@@
 			)
 		)
-		(model "${SPEAR_PCB_2026_DIR}/SPEAR_3D_Models/SPEAR_Motor_Controller_Carrier_Board/mill-max-4637-0-00-15-00-00-03-0.step"
+		(model "${SPEAR_PCB_2026_DIR}/SPEAR_3D_Models/SPEAR_MotorControllerCarrier/mill-max-4637-0-00-15-00-00-03-0.step"
 			(offset
 				(xyz 29.1 -13.9 14.6)
@@
 			)
 		)
-		(model "${SPEAR_PCB_2026_DIR}/SPEAR_3D_Models/SPEAR_Motor_Controller_Carrier_Board/mill-max-4637-0-00-15-00-00-03-0.step"
+		(model "${SPEAR_PCB_2026_DIR}/SPEAR_3D_Models/SPEAR_MotorControllerCarrier/mill-max-4637-0-00-15-00-00-03-0.step"
 			(offset
 				(xyz 29.1 -19 14.6)
@@
 			)
 		)
-		(model "${SPEAR_PCB_2026_DIR}/SPEAR_3D_Models/SPEAR_Motor_Controller_Carrier_Board/mill-max-0301-1-15-01-47-XX-10-0.step"
+		(model "${SPEAR_PCB_2026_DIR}/SPEAR_3D_Models/SPEAR_MotorControllerCarrier/mill-max-0301-1-15-01-47-XX-10-0.step"
 			(offset
 				(xyz 29.18 -1.25 9)
@@
 			)
 		)
-		(model "${SPEAR_PCB_2026_DIR}/SPEAR_3D_Models/SPEAR_Motor_Controller_Carrier_Board/mill-max-0301-1-15-01-47-XX-10-0.step"
+		(model "${SPEAR_PCB_2026_DIR}/SPEAR_3D_Models/SPEAR_MotorControllerCarrier/mill-max-0301-1-15-01-47-XX-10-0.step"
 			(offset
 				(xyz 29.18 -6.3 9)
@@
 			)
 		)
-		(model "${SPEAR_PCB_2026_DIR}/SPEAR_3D_Models/SPEAR_Motor_Controller_Carrier_Board/mill-max-0301-1-15-01-47-XX-10-0.step"
+		(model "${SPEAR_PCB_2026_DIR}/SPEAR_3D_Models/SPEAR_MotorControllerCarrier/mill-max-0301-1-15-01-47-XX-10-0.step"
 			(offset
 				(xyz 29.18 -13.95 9)
@@
 			)
 		)
-		(model "${SPEAR_PCB_2026_DIR}/SPEAR_3D_Models/SPEAR_Motor_Controller_Carrier_Board/mill-max-0301-1-15-01-47-XX-10-0.step"
+		(model "${SPEAR_PCB_2026_DIR}/SPEAR_3D_Models/SPEAR_MotorControllerCarrier/mill-max-0301-1-15-01-47-XX-10-0.step"
 			(offset
 				(xyz 29.18 -19 9)
@@
 		)
 	)
-	(footprint "Motor_Controller_Carrier_Board:FUSE_3557-10"
+	(footprint "SPEAR_MotorControllerCarrier:FUSE_3557-10"
 		(layer "F.Cu")
 		(at 144.675 79.724442 90)
@@
 		)
 		(embedded_fonts no)
-		(model "${SPEAR_PCB_2026_DIR}/SPEAR_3D_Models/SPEAR_Motor_Controller_Carrier_Board/3557-10.step"
+		(model "${SPEAR_PCB_2026_DIR}/SPEAR_3D_Models/SPEAR_MotorControllerCarrier/3557-10.step"
 			(offset
 				(xyz -0.4 0.15 4.5)
@@
 		)
 		(embedded_fonts no)
-		(model "${SPEAR_PCB_2026_DIR}/SPEAR_3D_Models/SPEAR_Motor_Controller_Carrier_Board/XT30PW-M.stp"
+		(model "${SPEAR_PCB_2026_DIR}/SPEAR_3D_Models/SPEAR_MotorControllerCarrier/XT30PW-M.stp"
 			(offset
 				(xyz -2.5 4.1 2.5)
@@
 		)
 	)
-	(footprint "Motor_Controller_Carrier_Board:CAP_UBY_18X20_NCH"
+	(footprint "SPEAR_MotorControllerCarrier:CAP_UBY_18X20_NCH"
 		(layer "F.Cu")
 		(at 179.375 88.306192 -90)
@@
 		)
 		(embedded_fonts no)
-		(model "${SPEAR_PCB_2026_DIR}/SPEAR_3D_Models/SPEAR_Motor_Controller_Carrier_Board/CAP_UBY_18X20_NCH.step"
+		(model "${SPEAR_PCB_2026_DIR}/SPEAR_3D_Models/SPEAR_MotorControllerCarrier/CAP_UBY_18X20_NCH.step"
 			(offset
 				(xyz 0 0 0)
@@
 		)
 	)
-	(footprint "Motor_Controller_Carrier_Board:CAP_C3225X7R1C226M250AC"
+	(footprint "SPEAR_MotorControllerCarrier:CAP_C3225X7R1C226M250AC"
 		(layer "F.Cu")
 		(at 123.5 100.23675 180)
@@
 		)
 		(embedded_fonts no)
-		(model "${SPEAR_PCB_2026_DIR}/SPEAR_3D_Models/SPEAR_Motor_Controller_Carrier_Board/C3225X7R1C226M250AC.step"
+		(model "${SPEAR_PCB_2026_DIR}/SPEAR_3D_Models/SPEAR_MotorControllerCarrier/C3225X7R1C226M250AC.step"
 			(offset
 				(xyz 0 -1.4 1.25)
@@
 		)
 	)
-	(footprint "Motor_Controller_Carrier_Board:CAPC3225X270N"
+	(footprint "SPEAR_MotorControllerCarrier:CAPC3225X270N"
 		(layer "F.Cu")
 		(at 113.75 97.23675)
@@
 		)
 		(embedded_fonts no)
-		(model "${SPEAR_PCB_2026_DIR}/SPEAR_3D_Models/SPEAR_Motor_Controller_Carrier_Board/GCM32EC71H106KA03L.step"
+		(model "${SPEAR_PCB_2026_DIR}/SPEAR_3D_Models/SPEAR_MotorControllerCarrier/GCM32EC71H106KA03L.step"
 			(offset
 				(xyz 0 -1.35 1.3)
@@
 		)
 		(embedded_fonts no)
-		(model "${SPEAR_PCB_2026_DIR}/SPEAR_3D_Models/SPEAR_Motor_Controller_Carrier_Board/XT30PW-M.stp"
+		(model "${SPEAR_PCB_2026_DIR}/SPEAR_3D_Models/SPEAR_MotorControllerCarrier/XT30PW-M.stp"
 			(offset
 				(xyz -2.5 4.1 2.5)
@@
 		)
 	)
-	(footprint "Motor_Controller_Carrier_Board:FUSE_3557-15"
+	(footprint "SPEAR_MotorControllerCarrier:FUSE_3557-15"
 		(layer "F.Cu")
 		(at 144.675 100.424442 -90)
@@
 		)
 		(embedded_fonts no)
-		(model "${SPEAR_PCB_2026_DIR}/SPEAR_3D_Models/SPEAR_Motor_Controller_Carrier_Board/3557-15.step"
+		(model "${SPEAR_PCB_2026_DIR}/SPEAR_3D_Models/SPEAR_MotorControllerCarrier/3557-15.step"
 			(offset
 				(xyz -0.4 0.15 4.5)
@@
 		)
 	)
-	(footprint "Motor_Controller_Carrier_Board:CAP_CC1206_YAG"
+	(footprint "SPEAR_MotorControllerCarrier:CAP_CC1206_YAG"
 		(layer "F.Cu")
 		(at 113.5 88.43735 -90)
@@
 		)
 		(embedded_fonts no)
-		(model "${SPEAR_PCB_2026_DIR}/SPEAR_3D_Models/SPEAR_Motor_Controller_Carrier_Board/CAP_CC1206_YAG.step"
+		(model "${SPEAR_PCB_2026_DIR}/SPEAR_3D_Models/SPEAR_MotorControllerCarrier/CAP_CC1206_YAG.step"
 			(offset
 				(xyz 0 0 0)
@@
 		)
 	)
-	(footprint "Motor_Controller_Carrier_Board:CAP_C3225X7R1C226M250AC"
+	(footprint "SPEAR_MotorControllerCarrier:CAP_C3225X7R1C226M250AC"
 		(layer "F.Cu")
 		(at 123.5 96.48675 180)
@@
 		)
 		(embedded_fonts no)
-		(model "${SPEAR_PCB_2026_DIR}/SPEAR_3D_Models/SPEAR_Motor_Controller_Carrier_Board/C3225X7R1C226M250AC.step"
+		(model "${SPEAR_PCB_2026_DIR}/SPEAR_3D_Models/SPEAR_MotorControllerCarrier/C3225X7R1C226M250AC.step"
 			(offset
 				(xyz 0 -1.4 1.25)
