File: SPEAR_PCB_Designs/DriveControllerCarrier/board_connectors.kicad_sch (KiCad schematic)
At the start: 9 parts, among them J10 Conn_01x01_Socket, J11 Conn_01x01_Socket, J5 Conn_01x20_Socket, J6 Conn_01x20_Socket, J7 Conn_01x08_Socket, J8 Conn_01x01_Socket, J9 Conn_01x01_Socket

Commit message: Routed traces for unconnected pins on stepper motor driver and did some organizing
Parts:
- J10, J11, J8, J9: symbol Motor_Controller_Carrier_Board:Conn_01x01_Socket_Flipped -> DriveControllerCarrier:Conn_01x01_Socket_Flipped
- J5, J6: symbol Motor_Controller_Carrier_Board:Conn_01x20_Socket_Flipped -> DriveControllerCarrier:Conn_01x20_Socket_Flipped
- J7: symbol Motor_Controller_Carrier_Board:Conn_01x08_Socket_Flipped -> DriveControllerCarrier:Conn_01x08_Socket_Flipped
Changed lines of the file:
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@@
 	)
 	(symbol
-		(lib_id "Motor_Controller_Carrier_Board:PWR_FLAG_Inline")
+		(lib_id "DriveControllerCarrier:PWR_FLAG_Inline")
 		(at 71.12 77.47 0)
 		(unit 1)
@@
 	)
 	(symbol
-		(lib_id "Motor_Controller_Carrier_Board:Conn_01x01_Socket_Flipped")
+		(lib_id "DriveControllerCarrier:Conn_01x01_Socket_Flipped")
 		(at 218.44 100.33 180)
 		(unit 1)
@@
 	)
 	(symbol
-		(lib_id "Motor_Controller_Carrier_Board:PWR_FLAG_Inline")
+		(lib_id "DriveControllerCarrier:PWR_FLAG_Inline")
 		(at 71.12 72.39 0)
 		(unit 1)
@@
 	)
 	(symbol
-		(lib_id "Motor_Controller_Carrier_Board:Conn_01x01_Socket_Flipped")
+		(lib_id "DriveControllerCarrier:Conn_01x01_Socket_Flipped")
 		(at 218.44 90.17 180)
 		(unit 1)
@@
 	)
 	(symbol
-		(lib_id "Motor_Controller_Carrier_Board:PWR_FLAG_Inline")
+		(lib_id "DriveControllerCarrier:PWR_FLAG_Inline")
 		(at 189.23 83.82 0)
 		(unit 1)
@@
 	)
 	(symbol
-		(lib_id "Motor_Controller_Carrier_Board:Conn_01x20_Socket_Flipped")
+		(lib_id "DriveControllerCarrier:Conn_01x20_Socket_Flipped")
 		(at 69.85 92.71 0)
 		(unit 1)
@@
 	)
 	(symbol
-		(lib_id "Motor_Controller_Carrier_Board:Conn_01x20_Socket_Flipped")
+		(lib_id "DriveControllerCarrier:Conn_01x20_Socket_Flipped")
 		(at 118.11 92.71 0)
 		(mirror y)
@@
 	)
 	(symbol
-		(lib_id "Motor_Controller_Carrier_Board:PWR_FLAG_Inline")
+		(lib_id "DriveControllerCarrier:PWR_FLAG_Inline")
 		(at 71.12 74.93 0)
 		(unit 1)
@@
 	)
 	(symbol
-		(lib_id "Motor_Controller_Carrier_Board:PWR_FLAG_Inline")
+		(lib_id "DriveControllerCarrier:PWR_FLAG_Inline")
 		(at 217.17 85.09 0)
 		(unit 1)
@@
 	)
 	(symbol
-		(lib_id "Motor_Controller_Carrier_Board:Conn_01x01_Socket_Flipped")
+		(lib_id "DriveControllerCarrier:Conn_01x01_Socket_Flipped")
 		(at 218.44 85.09 180)
 		(unit 1)
@@
 	)
 	(symbol
-		(lib_id "Motor_Controller_Carrier_Board:Conn_01x08_Socket_Flipped")
+		(lib_id "DriveControllerCarrier:Conn_01x08_Socket_Flipped")
 		(at 187.96 91.44 0)
 		(unit 1)
@@
 	)
 	(symbol
-		(lib_id "Motor_Controller_Carrier_Board:PWR_FLAG_Inline")
+		(lib_id "DriveControllerCarrier:PWR_FLAG_Inline")
 		(at 71.12 69.85 0)
 		(unit 1)
@@
 	)
 	(symbol
-		(lib_id "Motor_Controller_Carrier_Board:Conn_01x01_Socket_Flipped")
+		(lib_id "DriveControllerCarrier:Conn_01x01_Socket_Flipped")
 		(at 218.44 95.25 180)
 		(unit 1)
@@
 	)
 	(symbol
-		(lib_id "Motor_Controller_Carrier_Board:PWR_FLAG_Inline")
+		(lib_id "DriveControllerCarrier:PWR_FLAG_Inline")
 		(at 217.17 100.33 0)
 		(unit 1)
