File: SPEAR_PCB_Designs/EtherCatDevBoard_V1-1/EtherCatDevBoard_V1-1.kicad_sch (KiCad schematic)
At the start: 0 parts

Commit message: Updates to V1.1 for Ecat dev board.
Other:
- sheet LAN9252 ports: added SCS; removed CS
Changed lines of the file:
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@@
 		)
 		(instances
-			(project "SPEAR_V1"
+			(project "EtherCatDevBoard_V1-1"
 				(path "/6af343d7-7346-4b6a-90ee-eb113982f4e5"
 					(page "2")
@@
 			)
 		)
-		(pin "CS" input
-			(at 71.12 59.69 180)
-			(effects
-				(font
-					(size 1.27 1.27)
-				)
-				(justify left)
-			)
-		)
 		(pin "IRQ" output
 			(at 71.12 63.5 180)
@@
 			)
 		)
+		(pin "SCS" input
+			(at 71.12 59.69 180)
+			(effects
+				(font
+					(size 1.27 1.27)
+				)
+				(justify left)
+			)
+		)
 		(instances
-			(project "SPEAR_V1"
+			(project "EtherCatDevBoard_V1-1"
 				(path "/6af343d7-7346-4b6a-90ee-eb113982f4e5"
 					(page "3")
