File: SPEAR_PCB_Designs/EtherCatDevBoard_V1-1/lan9252.kicad_sch (KiCad schematic)
At the start: 29 parts, among them U4 LAN9252I/ML, Y2 25MHz

Commit message: Updates to V1.1 for Ecat dev board.
Connections:
- net SCS: now reaches U4.50 (D5)
- net CS: no longer names the net of U4.28 (CS)
Changed lines of the file:
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@@
 	)
 	(no_connect
+		(at 85.09 115.57)
+	)
+	(no_connect
 		(at 85.09 120.65)
 	)
@@
 	)
 	(no_connect
-		(at 156.21 118.11)
-	)
-	(no_connect
 		(at 156.21 123.19)
 	)
@@
 	(wire
 		(pts
-			(xy 78.74 115.57) (xy 85.09 115.57)
-		)
-		(stroke
-			(width 0)
-			(type default)
-		)
-	)
-	(wire
-		(pts
 			(xy 275.59 55.88) (xy 275.59 60.96)
 		)
@@
 	(wire
 		(pts
+			(xy 165.1 118.11) (xy 156.21 118.11)
+		)
+		(stroke
+			(width 0)
+			(type default)
+		)
+	)
+	(wire
+		(pts
 			(xy 60.96 99.06) (xy 49.53 99.06)
 		)
@@
 		)
 	)
-	(hierarchical_label "CS"
+	(hierarchical_label "SCS"
 		(shape input)
-		(at 78.74 115.57 180)
+		(at 165.1 118.11 0)
 		(effects
 			(font
 				(size 1.27 1.27)
 			)
-			(justify right)
+			(justify left)
 		)
 	)
@@
 		)
 		(instances
-			(project "SPEAR_V1"
+			(project "EtherCatDevBoard_V1-1"
 				(path "/6af343d7-7346-4b6a-90ee-eb113982f4e5/d630782a-bbb8-450e-a52a-35375a587c4e"
 					(page "4")
