File: SPEAR_PCB_Designs/EtherCatDevBoard_V1-1/stm32f446rc.kicad_sch (KiCad schematic)
At the start: 39 parts, among them J1 USB_C_Receptacle_USB2.0_16P, J2 FTSH-107-01-F-DV-K-P-TR, J3 Conn_01x20_Pin, J4 Conn_01x20_Pin, SW1 SW_Push, U1 USBLC6-2SC6, U2 STM32F446RCT6, U3 AMS1117-3.3 SOT-223, U6 TPS2116DRL, Y1 16MHz

Commit message: Updates to V1.1 for Ecat dev board.
Parts:
- Y1: footprint Crystal:Crystal_SMD_3225-4Pin_3.2x2.5mm -> Crystal:Crystal_SMD_2520-4Pin_2.5x2.0mm
Changed lines of the file:
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@@
 			)
 		)
-		(property "Footprint" "Crystal:Crystal_SMD_3225-4Pin_3.2x2.5mm"
+		(property "Footprint" "Crystal:Crystal_SMD_2520-4Pin_2.5x2.0mm"
 			(at 85.09 68.58 0)
 			(effects
