File: SPEAR_PCB_Designs/BMS_Carrier_Board/BMS Carrier Board.kicad_pcb (KiCad board)
At the start: 4 copper layers, 38 parts, among them J1 B4B-XH-A, J2 B10B-XH-A, J3 B2B-XH-A, J4 B7B-XH-A, J5 B2B-XH-A, J6 B2B-XH-A, J7 B2B-XH-A, J8 Conn_01x02_Pin, U1 AP63203WU, U6 TPS2116DRL

Commit message: BMS Carrier Board done
Parts:
- removed C15: 22uF, Capacitor_SMD:C_0805_2012Metric
- removed F10: C1Q 1.5, BMS footprints:C1_BEL
- removed F12: 2A, SPEAR_MotorControllerCarrier:FUS_LITTELFUSE_392_LTF
- removed R3, R4: 5.1kR, Resistor_SMD:R_0402_1005Metric
- added F9: C1Q 1.5, BMS footprints:C1_BEL, F.Cu at (41.4, 62.0)
- added J10: B2B-XH-A, BMS footprints:CONN_B2B-XH-A_JST, F.Cu at (97.0, 27.2)
- added J9: SM02B-GHS-TB, BMS footprints:CONN_SM02B-GHS_JST, F.Cu at (96.8, 70.7)
- added R1: CT-6EP103, BMS footprints:POT_CT-6EP103_NDC, F.Cu at (67.5, 40.2)
- J2: value B10B-XH-A -> B16B-PHDSS; footprint BMS footprints:CONN_B10B-XH-A_JST -> BMS footprints:CONN16_B16B-PHDSS_JST
- J8: value Conn_01x02_Pin -> B9B-XH-A LFSN; footprint SPEAR_Connectors:AMASS_XT30PW-M_1x02_P2.50mm_Horizontal_1 -> BMS footprints:CONN_B9B-XH-A_JST
- U1: footprint SPEAR_MotorControllerCarrier:TSOT-23-6 -> Package_TO_SOT_SMD:TSOT-23-6
- moved J2 157.2 mm to (64.0, 29.2), turned to 180 degrees
- moved C1 152.2 mm to (48.8, 62.2)
- moved C2 152.2 mm to (48.8, 66.0)
- moved C3 152.2 mm to (48.5, 53.4)
- moved C4 152.2 mm to (58.5, 65.2)
- moved C5 152.2 mm to (58.5, 61.5)
- moved L1 152.2 mm to (58.0, 53.7)
- moved U1 152.2 mm to (48.5, 58.2)
- moved J3 143.7 mm to (31.2, 29.7), turned to 90 degrees
- moved F7 137.1 mm to (41.4, 40.7)
- moved J7 136.2 mm to (31.2, 67.7), turned to 90 degrees
- moved J6 133.4 mm to (31.2, 59.2), turned to 90 degrees
- moved F6 132.3 mm to (41.4, 43.2)
- moved F5 127.7 mm to (41.4, 45.7)
- moved F4 123.1 mm to (41.4, 48.2)
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Connections:
- net /STM32F446RC/PWR_LED_K renamed /PWR_LED_K
- net /Schematic/BST renamed /BST
- net /Schematic/BUCK_PWR renamed /BUCK_PWR
- net /Schematic/SW renamed /SW
- C50 pad 1: /STM32F446RC/3.3V_USB -> /3.3V_BMS
- C51 pad 1: /STM32F446RC/3.3V_Battery -> /3.3V_Battery
- J1 pad 4: Net-(J1-Pad4) -> GND
- J2 pad 1: unconnected-(J2-Pad1) -> GND
- J2 pad 10: Net-(J2-Pad10) -> Net-(MCB1-PB5)
- J2 pad 2: unconnected-(J2-Pad2) -> Net-(MCB1-+3.3V)
- J2 pad 3: Net-(F7-Pad2) -> Net-(J2-Pad3)
- J2 pad 4: Net-(F6-Pad2) -> Net-(MCB1-PA15)
- J2 pad 5: Net-(F5-Pad2) -> Net-(MCB1-PC10)
- J2 pad 6: Net-(F4-Pad2) -> Net-(MCB1-PC11)
- J2 pad 7: Net-(F3-Pad2) -> Net-(MCB1-PC12)
- J2 pad 8: Net-(F2-Pad2) -> Net-(MCB1-PD2)
- J2 pad 9: Net-(F1-Pad2) -> Net-(MCB1-PB4)
- J3 pad 1: Net-(J2-Pad10) -> Net-(J10-Pad2)
- J6 pad 2: Net-(J5-Pad1) -> GND
- J8 pad 1: GND -> unconnected-(J8-Pad1)
- J8 pad 2: Net-(J1-Pin_2) -> unconnected-(J8-Pad2)
- MCB1 pad 10: unconnected-(MCB1-PC11-Pad10) -> Net-(MCB1-PC11)
- MCB1 pad 11: unconnected-(MCB1-PC12-Pad11) -> Net-(MCB1-PC12)
- MCB1 pad 12: unconnected-(MCB1-PD2-Pad12) -> Net-(MCB1-PD2)
- MCB1 pad 13: unconnected-(MCB1-PB4-Pad13) -> Net-(MCB1-PB4)
- MCB1 pad 14: unconnected-(MCB1-PB5-Pad14) -> Net-(MCB1-PB5)
- MCB1 pad 15: unconnected-(MCB1-PB6-Pad15) -> Net-(MCB1-PB6)
- MCB1 pad 16: unconnected-(MCB1-PB7-Pad16) -> Net-(MCB1-PB7)
- MCB1 pad 17: unconnected-(MCB1-PB8-Pad17) -> Net-(MCB1-PB8)
- MCB1 pad 18: unconnected-(MCB1-PB9-Pad18) -> Net-(MCB1-PB9)
- MCB1 pad 2: unconnected-(MCB1-GND-Pad2) -> GND
- MCB1 pad 3: unconnected-(MCB1-+3.3V-Pad3) -> Net-(MCB1-+3.3V)
- MCB1 pad 4: Net-(J1-Pad4) -> GND
- MCB1 pad 8: unconnected-(MCB1-PA15-Pad8) -> Net-(MCB1-PA15)
- MCB1 pad 9: unconnected-(MCB1-PC10-Pad9) -> Net-(MCB1-PC10)
- R32 pad 2: /STM32F446RC/3.3V_USB -> /3.3V_BMS
- U6 pad 3: /STM32F446RC/3.3V_USB -> /3.3V_BMS
- U6 pad 5: /STM32F446RC/3.3V_USB -> /3.3V_BMS
- U6 pad 6: /STM32F446RC/3.3V_Battery -> /3.3V_Battery
Routing:
- net +3.3V: track 7.53 -> 111.6 mm, vias 3 -> 2
- net Net-(F1-Pad2): track 0.00 -> 93.6 mm, vias 0 -> 1
- net Net-(F8-Pad2): track 0.00 -> 79.6 mm
- net Net-(J10-Pad2): track 0.00 -> 69.3 mm
- net Net-(F7-Pad2): track 0.00 -> 55.0 mm, vias 0 -> 1
- net Net-(F6-Pad2): track 0.00 -> 54.2 mm, vias 0 -> 1
- net Net-(F5-Pad2): track 0.00 -> 54.2 mm, vias 0 -> 1
- net Net-(F4-Pad2): track 0.00 -> 54.2 mm, vias 0 -> 1
- net Net-(F3-Pad2): track 0.00 -> 54.2 mm, vias 0 -> 1
- net Net-(F2-Pad2): track 0.00 -> 54.2 mm, vias 0 -> 1
- net /3.3V_BMS: track 0.00 -> 53.6 mm
- net Net-(MCB1-+3.3V): track 0.00 -> 31.8 mm
- net /3.3V_Battery: track 53.6 -> 26.1 mm
- net Net-(F8-Pad1): track 0.00 -> 26.5 mm
- net Net-(J5-Pad2): track 0.00 -> 14.6 mm
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- added copper zone on B.Cu, net GND
- removed copper zone on In2.Cu, net +3.3V
- removed copper zone on In1.Cu, net GND
Other:
- board outline added: 73.2 x 53 mm
- copper layers 4 -> 2
- board text added: "David Stobbe"
- board text removed: "BATT IN"
- board text removed: "BATT OUT"
- board text removed: "OUT"
