File: SPEAR_PCB_Designs/BMS_Carrier_Board/BMS Carrier Board.kicad_sch (KiCad schematic)
At the start: 35 parts, among them J1 B4B-XH-A, J2 B2B-XH-A, J3 B2B-XH-A, J4 B7B-XH-A, J5 B2B-XH-A, J6 B2B-XH-A, J7 B2B-XH-A, J8 B9B-XH-A LFSN, J9 SM02B-GHS-TB, U1 AP63203WU, U6 TPS2116DRL

Commit message: BMS Carrier Board done
Parts:
- removed J2: B2B-XH-A, CONN_B2B-XH-A_JST, symbol BMS symbols:B2B-XH-A
- added J10: B2B-XH-A, CONN_B2B-XH-A_JST, symbol BMS symbols:B2B-XH-A
- added J2: B16B-PHDSS, CONN16_B16B-PHDSS_JST, symbol BMS symbols:B16B-PHDSS
- added R1: CT-6EP103, POT_CT-6EP103_NDC, symbol BMS symbols:CT-6EP103
- J8: footprint CONN_B9B-XH-ALFSN_JST -> CONN_B9B-XH-A_JST
Connections:
- net GND: now also J1.4, J6.2, MCB1.2 (GND), MCB1.4 (GND), J10.1, J2.1, J2.15, J2.16, R1.1
- net at J3.1: now also J10.2
- net at MCB1.10 (PC11): now also J2.6
- net at MCB1.11 (PC12): now also J2.7
- net at MCB1.12 (PD2): now also J2.8
- net at MCB1.13 (PB4): now also J2.9
- net at MCB1.14 (PB5): now also J2.10
- net at MCB1.15 (PB6): now also J2.11
- net at MCB1.16 (PB7): now also J2.12
- net at MCB1.17 (PB8): now also J2.13
- net at MCB1.18 (PB9): now also J2.14
- net at MCB1.3 (+3.3V): now also J2.2, R1.3
- net at MCB1.8 (PA15): now also J2.4
- net at MCB1.9 (PC10): now also J2.5
- net at J5.1: now also J9.1; no longer J9.2
- net at J5.2: now also J9.2; no longer J9.1
- new net: J2.3, R1.2
- no-connect marks 4 -> 23
Other:
- moved on the sheet: F8, F9, J1, J6, J7, J9, MCB1
