File: SPEAR_PCB_Designs/LAN9252_Junction/LAN9252_Junction.kicad_sch (KiCad schematic)
At the start: 2 parts

Commit message: Fixed this finally
Other:
- sheet Buck Converter: file C:/Users/sheeb/OneDrive/Documents/IGuessThisIsTheFinalBoard(s)/pcb_designs_2026/SPEAR_PCB_Designs/AP63203BuckConverter/AP63203BuckConverter.kicad_sch -> ../AP63203BuckConverter/AP63203BuckConverter.kicad_sch
Changed lines of the file:
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@@
 			)
 		)
-		(property "Sheetfile" "C:/Users/sheeb/OneDrive/Documents/IGuessThisIsTheFinalBoard(s)/pcb_designs_2026/SPEAR_PCB_Designs/AP63203BuckConverter/AP63203BuckConverter.kicad_sch"
+		(property "Sheetfile" "../AP63203BuckConverter/AP63203BuckConverter.kicad_sch"
 			(at 201.93 116.1546 0)
 			(effects
